File: temp_display.sch (EAGLE design)
At the start: 71 parts, among them IC2 ATMEGA168PROUND, Q1 2N2907, Q2 FQN1N50C, T1 BC547

Commit message: Fixed some shorts. Now need to align indicators and code (wrong LEDs light up)
Parts:
- removed Q2: FQN1N50C, adafruit:FQN1N50C
- added H1, H2, H3: MOUNT-PAD-ROUND3.0, holes:MOUNT-PAD-ROUND3.0
- added U$3: 2N7000, kirill:2N7000
- R8, R9: device resistor:R-US_0204/7 -> resistor:R-US_0204/2V
Connections:
- removed net +5: C1.+, C2.2, C3.1, IC1.IN, IC2.AVCC, IC2.VCC, JP1.2, JP9.11, JP9.15, JP9.19, JP9.23, JP9.3, JP9.7, POWER_SW.2, Q1.E, R31.1, SR2.MR, SR2.VCC, U$6.9
- new net N$16: JP8.1, POWER_SW.1
- net +5V: now also C1.+, C2.2, C3.1, IC1.IN, IC2.AVCC, IC2.VCC, JP1.2, JP9.11, JP9.15, JP9.19, JP9.23, JP9.3, JP9.7, POWER_SW.2, Q1.E, R31.1, SR2.MR, SR2.VCC, U$6.9; no longer JP8.1, POWER_SW.1
- net GND: now also U$3.S; no longer Q2.S
- net N$14: now also U$3.G; no longer Q2.G
- net OE: now also U$3.D; no longer Q2.D
Other:
- moved on the sheet: R9
